File: src/issue3b.kicad_sch (KiCad schematic)
At the start: 0 parts

Commit message: Added R25 to BOM Started Schematic
Parts:
- added C1, C2, C26, C29, C3, C30, C33, C4, C40, C41, C42, C48, C5, C55, C56, C57, C58, C59, C6, C60, C61, C62, C66, C7, C76, C8: 47nF, symbol Device:C_Small
- added C25, C28, C34, C47, C50, C65: 22uF, Capacitor_THT:CP_Axial_L11.0mm_D6.0mm_P18.00mm_Horizontal, symbol Issue 4-rescue:CP_Small-Device
- added C27, C46: 1uF, Capacitor_THT:CP_Axial_L11.0mm_D6.0mm_P18.00mm_Horizontal, symbol Issue 4-rescue:CP_Small-Device
- added C31, C32, C43, C68, C69, C70, C71, C75, C77: 100nF, symbol Device:C_Small
- added C35, C39: 10nF, symbol Device:C_Small
- added C37, C38: 33pF, symbol Device:C_Small
- added C44, C45: 100uF, Capacitor_THT:CP_Axial_L11.0mm_D6.0mm_P18.00mm_Horizontal, symbol Issue 4-rescue:CP_Small-Device
- added C49: 560pF, symbol Device:C_Small
- added C52, C53: 150pF, symbol Device:C_Small
- added C64, C67: 100pF, symbol Device:C_Small
- added C72, C73: 16pF, symbol Device:C_Small
- added C74: 4.7uF, Capacitor_THT:CP_Axial_L11.0mm_D6.0mm_P18.00mm_Horizontal, symbol Issue 4-rescue:CP_Small-Device
- added D1, D11, D13, D18, D2, D3, D4, D5, D6, D7, D8, D9: 1N4148, symbol Diode:1N4148
- added D15: BA157, symbol Diode:1N4148
- added D19: DZY88, Diode_THT:D_DO-35_SOD27_P7.62mm_Horizontal, symbol Device:D_Zener
- added E1: Edge_Connector, symbol Issue-4-rescue:Edge_Connector-spectrum
- added Ear0, Mic0: Barrel_Jack, symbol Connector:Barrel_Jack
- added IC1: ULA, Package_DIP:DIP-40_W15.24mm_Socket, symbol Issue-4-rescue:ULA-spectrum
- added IC10, IC11, IC12, IC13, IC6, IC7, IC8, IC9: 4116, Package_DIP:DIP-16_W7.62mm_Socket, symbol Issue-4-rescue:4116-spectrum
- added IC14: LM1889, Package_DIP:DIP-18_W7.62mm_Socket, symbol Issue-4-rescue:LM1809-spectrum
- added IC15, IC16, IC17, IC18, IC19, IC20, IC21, IC22: 4532, Package_DIP:DIP-16_W7.62mm_Socket, symbol Issue-4-rescue:4532-spectrum
- added IC2: Z80, Package_DIP:DIP-40_W15.24mm_Socket, symbol Issue-4-rescue:Z80-spectrum
- added IC23: 74LS32, Package_DIP:DIP-14_W7.62mm_Socket, symbol 74xx:74LS32
- added IC24: 74LS00, Package_DIP:DIP-14_W7.62mm_Socket, symbol 74xx:74LS00
- added IC25, IC26: 74LS157, Package_DIP:DIP-16_W7.62mm_Socket, symbol Issue-4-rescue:74LS157-spectrum
- added IC3: 74LS157, Package_DIP:DIP-16_W7.62mm_Socket, symbol Issue-4-rescue:LS157-spectrum
- added IC4: 74LS157, Package_DIP:DIP-16_W7.62mm_Socket, symbol Issue-4-rescue:LS157-A-spectrum
- added IC5: ROM, Package_DIP:DIP-28_W15.24mm_Socket, symbol Issue-4-rescue:ROM-spectrum
- added J1: OKI, Connector_PinHeader_2.54mm:PinHeader_1x03_P2.54mm_Vertical, symbol Connector_Generic:Conn_01x03
- added J10: UR3, Connector_PinHeader_2.54mm:PinHeader_1x01_P2.54mm_Vertical, symbol Connector_Generic:Conn_01x01
- added J11: UR4, Connector_PinHeader_2.54mm:PinHeader_1x01_P2.54mm_Vertical, symbol Connector_Generic:Conn_01x01
- added J2, J3, J4: TI, Connector_PinHeader_2.54mm:PinHeader_1x03_P2.54mm_Vertical, symbol Connector_Generic:Conn_01x03
- added J7: Barrel_Jack_MountingPin, symbol Connector:Barrel_Jack_MountingPin
- added J8: UR1, Connector_PinHeader_2.54mm:PinHeader_1x01_P2.54mm_Vertical, symbol Connector_Generic:Conn_01x01
- added J9: UR2, Connector_PinHeader_2.54mm:PinHeader_1x01_P2.54mm_Vertical, symbol Connector_Generic:Conn_01x01
- added KB1: Conn_01x05, Connector_PinSocket_2.54mm:PinSocket_1x05_P2.54mm_Vertical, symbol Connector_Generic:Conn_01x05
- added KB2: Conn_01x08, Connector_PinSocket_2.54mm:PinSocket_1x08_P2.54mm_Vertical, symbol Connector_Generic:Conn_01x08
- added LS1: Speaker, symbol Device:Speaker
- added R1, R2, R26, R27, R3, R4, R5, R6, R7, R78, R8: 470, symbol Device:R
- added R10, R11, R12, R13, R14, R15, R16, R9: 8k2, symbol Device:R
- added R17, R18, R19, R20, R21, R22, R23: 330, symbol Device:R
- added R24, R37, R42, R45, R46, R47, R56, R63, R73, R76, R77: 1K, symbol Device:R
- added R28, R29, R30, R35, R49, R65, R66, R67, R68, R69, R72, R74, R75: 10K, symbol Device:R
- added R31: 220K, symbol Device:R
- added R32: 100, symbol Device:R
- added R33, R36: 680, symbol Device:R
- added R34: 15 1W, Resistor_THT:R_Axial_Power_L20.0mm_W6.4mm_P22.40mm, symbol Device:R
- added R43: 3K, symbol Device:R
- added R44: 5K1, symbol Device:R
- added R48: 4K7, symbol Device:R
- added R50: 8K2, symbol Device:R
- added R51, R52: 2K2, symbol Device:R
- added R53: 390R, symbol Device:R
- added R58: 1K 2%, symbol Device:R
- added R59: 1K8 2%, symbol Device:R
- added R60: 68, symbol Device:R
- added R61, R62, R64: 15, symbol Device:R
- added R70, R71: 220, symbol Device:R
- added R79: 2k2, symbol Device:R
- added REG1: L7805, symbol Regulator_Linear:L7805
- added T1: Coil, symbol Device:Transformer_1P_1S
- added TR1, TR2, TR3, TR6: ZTX313, Package_TO_SOT_THT:TO-92Flat, symbol Transistor_BJT:BC547
- added TR4: ZTX650, Package_TO_SOT_THT:TO-92Flat, symbol Transistor_BJT:BC547
- added TR5: ZTX313, Package_TO_SOT_THT:TO-92Flat, symbol Device:Q_PNP_CBE
- added TR7: ZTX450, Package_TO_SOT_THT:TO-92Flat, symbol Transistor_BJT:BC547
- added TR8, TR9: BC184, Package_TO_SOT_THT:TO-92_Inline, symbol Transistor_BJT:BC547
- added TV1: Modulator, symbol Issue-4-rescue:Modulator
- added X1: 14Mhz, Crystal:Crystal_HC18-U_Vertical, symbol Device:Crystal
- added X2: 4.43Mhz, Crystal:Crystal_HC18-U_Horizontal, symbol Device:Crystal
Connections:
- new net: IC1.12 (_INT), R26.2
- new net: C30.2, IC1.13 (Vcc2), R34.2
- new net: IC1.18 (D0), IC6.14 (DOUT), IC6.2 (DIN), R1.2
- new net: IC1.19 (KB0), KB1.1 (Pin_1), R69.2
- new net: IC1.20 (KB1), KB1.2 (Pin_2), R68.2
- new net: IC1.21 (D1), IC7.14 (DOUT), IC7.2 (DIN), R2.2
- new net: IC1.22 (D2), IC8.14 (DOUT), IC8.2 (DIN), R3.2
- new net: IC1.23 (KB2), KB1.3 (Pin_3), R67.2
- new net: IC1.24 (KB3), KB1.4 (Pin_4), R66.2
- new net: IC1.25 (D3), IC9.14 (DOUT), IC9.2 (DIN), R4.2
- new net: IC1.26 (KB4), KB1.5 (Pin_5), R65.2
- new net: IC1.27 (D4), IC10.14 (DOUT), IC10.2 (DIN), R5.2
- new net: C32.1, C35.2, D13.1 (K), D9.2 (A), IC1.28 (MIC/TAPE), R35.2
- new net: IC1.29 (D5), IC11.14 (DOUT), IC11.2 (DIN), R6.2
- new net: IC1.30 (D6), IC12.14 (DOUT), IC12.2 (DIN), R7.2
- new net: IC1.31 (D7), IC13.14 (DOUT), IC13.2 (DIN), R8.2
- new net: IC1.34 (_ROMCS), R33.2
- new net: IC1.39 (OSC), X1.2
- new net: IC3.12 (4Y), R23.1
- new net: IC3.4 (1Y), R22.1
- new net: IC3.7 (2Y), R21.1
- new net: IC3.9 (3Y), R20.1
- new net: IC3.1 (S), IC4.1 (S), R32.1
- new net: IC4.12 (4Y), R19.1
- new net: IC4.4 (1Y), R18.1
- new net: IC4.7 (2Y), R17.1
- new net: C65.1, IC14.13 (CHROMA_SUB-CARRIER), R72.2
- new net: C65.2, R51.1, TR1.1 (C), TR2.2 (B)
- new net: IC5.20 (CS), J8.1 (Pin_1)
- new net: IC5.27 (OE1L), J11.1 (Pin_1)
- new net: C67.2, R24.1, TR3.2 (B)
- new net: C73.2, X1.1
- new net: C47.2, D15.2 (A)
- new net: D1.2 (A), KB2.1 (Pin_1)
- new net: D2.2 (A), KB2.2 (Pin_2)
- new net: D3.2 (A), KB2.3 (Pin_3)
- new net: D4.2 (A), KB2.4 (Pin_4)
- new net: D5.2 (A), KB2.5 (Pin_5)
- new net: D6.2 (A), KB2.6 (Pin_6)
- new net: D7.2 (A), KB2.7 (Pin_7)
- new net: D8.2 (A), KB2.8 (Pin_8)
- new net: D9.1 (K), TR7.2 (B)
- new net: LS1.2, TR7.3 (E)
- new net: C25.1, C40.1, C42.1, R49.2, R51.2, R64.1, R72.1, TR2.1 (C), TV1.1 (+5V)
- new net: C32.2, R36.2
- new net: Ear0.2, R36.1, R37.1
- new net: C31.1, R35.1
- new net: C31.2, Mic0.2
- new net: IC26.10 (3B), J1.1 (Pin_1), J1.2 (Pin_2), J1.3 (Pin_3)
- new net: C46.2, D11.2 (A), D18.1 (K)
- new net: C39.1, IC14.1 (CHROMA_LEAD)
- new net: IC14.12 (VIDEO_INPUT), R42.2
- new net: IC14.17 (CHROMA_OSC_OUTPUT), R43.2, R44.2
- new net: C37.1, IC14.18 (CHROMA_LAG), R45.2
- new net: C53.1, IC14.2 (R-Y_INPUT), R77.2
- new net: C76.2, IC14.3 (CHROMA_BIAS), R78.2
- new net: C52.1, IC14.4 (B-Y_INPUT), R76.2
- new net: D18.2 (A), R79.1
- new net: IC26.11 (3A), J2.1 (Pin_1), J2.2 (Pin_2), J2.3 (Pin_3)
- new net: C74.2, R58.1, R59.1, TR5.2 (B)
- new net: C71.1, R77.1, TR8.1 (C)
- new net: C70.1, R75.1, TR8.2 (B)
- new net: C69.1, R76.1, TR9.1 (C)
- new net: C68.1, R74.1, TR9.2 (B)
- new net: C72.1, R44.1, X2.1
- new net: C38.2, R45.1, X2.2
- new net: C38.1, C39.2, R46.2
- new net: R48.1, R49.1, R50.2, TR1.2 (B)
- new net: R52.2, TR1.3 (E)
- new net: IC23.8, IC25.1 (S), IC26.1 (S), R70.1
- new net: IC24.6, IC24.9
- new net: IC23.10, IC24.8
- new net: C64.1, IC23.5, R70.2
- new net: R60.1, TR5.1 (C)
- new net: C43.2, R60.2, R61.1
- new net: C77.2, R61.2, T1.1 (AA)
- new net: T1.2 (AB), TR4.2 (B)
- new net +12V: C44.1, C5.1, C6.1, C7.1, C8.1, D15.1 (K), E1.21, IC10.8 (VDD), IC11.8 (VDD), IC12.8 (VDD), IC13.8 (VDD), IC6.8 (VDD), IC7.8 (VDD), IC8.8 (VDD), IC9.8 (VDD), R59.2, R62.1
- new net +12VA: C33.2, C45.1, C48.2, C52.2, C53.2, IC14.14 (RF_SUPPLY), IC14.15 (SOUND_TANK), IC14.16 (CHROMA_SUPPLY), R42.1, R62.2
- new net +5V: C1.1, C1.2, C2.1, C2.2, C25.2, C26.1, C26.2, C27.2, C28.1, C28.2, C29.1, C29.2, C3.1, C3.2, C30.1, C33.1, C34.1, C34.2, C35.1, C37.2, C4.1, C4.2, C40.2, C41.1, C41.2, C42.2, C43.1, C44.2, C45.2, C48.1, C49.1, C5.2, C50.2, C55.1, C55.2, C56.1, C56.2, C57.1, C57.2, C58.1, C58.2, C59.1, C59.2, C6.2, C60.1, C60.2, C61.1, C61.2, C62.1, C62.2, C64.2, C66.1, C7.2, C72.2, C73.1, C74.1, C75.1, C75.2, C76.1, C77.1, C8.2, D11.1 (K), D13.2 (A), D19.1 (K), D19.2 (A), E1.19, E1.30, E1.32, E1.33, E1.40, Ear0.1, IC1.14 (Vcc1), IC1.40 (GND), IC10.1 (VBB), IC10.16 (VSS), IC10.9 (VCC), IC11.1 (VBB), IC11.16 (VSS), IC11.9 (VCC), IC12.1 (VBB), IC12.16 (VSS), IC12.9 (VCC), IC13.1 (VBB), IC13.16 (VSS), IC13.9 (VCC), IC14.5 (GROUND), IC15.1 (NC), IC15.16 (VSS), IC15.8 (VDD), IC16.1 (NC), IC16.16 (VSS), IC16.8 (VDD), IC17.1 (NC), IC17.16 (VSS), IC17.8 (VDD), IC18.1 (NC), IC18.16 (VSS), IC18.8 (VDD), IC19.1 (NC), IC19.16 (VSS), IC19.8 (VDD), IC2.11 (VCC), IC2.29 (GND), IC2.6 (~{CLK}), IC20.1 (NC), IC20.16 (VSS), IC20.8 (VDD), IC21.1 (NC), IC21.16 (VSS), IC21.8 (VDD), IC22.1 (NC), IC22.16 (VSS), IC22.8 (VDD), IC23.14 (VCC), IC23.7 (GND), IC23.9, IC24.14 (VCC), IC24.7 (GND), IC25.15 (STROBE), IC25.16 (VCC), IC25.8 (GND), IC26.15 (STROBE), IC26.16 (VCC), IC26.8 (GND), IC3.15 (STROBE), IC3.16 (VCC), IC3.8 (GND), IC4.15 (STROBE), IC4.16 (VCC), IC4.8 (GND), IC5.14 (Vss), IC5.28 (Vcc), IC6.1 (VBB), IC6.16 (VSS), IC6.9 (VCC), IC7.1 (VBB), IC7.16 (VSS), IC7.9 (VCC), IC8.1 (VBB), IC8.16 (VSS), IC8.9 (VCC), IC9.1 (VBB), IC9.16 (VSS), IC9.9 (VCC), J3.2 (Pin_2), J3.3 (Pin_3), J4.2 (Pin_2), J4.3 (Pin_3), J7.1, LS1.1, Mic0.1, R10.1, R11.1, R12.1, R13.1, R14.1, R15.1, R16.1, R28.1, R29.1, R30.1, R31.1, R34.1, R37.2, R43.1, R46.1, R47.1, R50.1, R52.1, R53.1, R56.2, R58.2, R63.2, R64.2, R65.1, R66.1, R67.1, R68.1, R69.1, R71.2, R73.1, R74.2, R75.2, R78.1, R79.2, R9.1, REG1.2 (GND), REG1.3 (OUT), TR3.1 (C), TR3.3 (E), TR4.3 (E), TR5.3 (E), TR6.1 (C), TR7.1 (C), TR8.3 (E), TR9.3 (E), TV1.3 (GND)
- new net +9V: C50.1, C66.2, E1.31, J7.2, J7.MP (MountPin), REG1.1 (IN), T1.4 (SB)
- new net -12V: C46.1, C47.1, C49.2, E1.22, T1.3 (SA), TR4.1 (C)
- new net A0: E1.35, IC2.30 (A8), IC26.6 (2B), IC4.6 (2B), IC5.10 (A0), TR6.2 (B)
- new net A1: E1.36, IC2.31 (A1), IC26.3 (1B), IC4.3 (1B), IC5.9 (A1)
- new net A10: D2.1 (K), E1.26, IC2.40 (A10), IC25.11 (3A), IC3.11 (3A), IC5.21 (A10)
- new net A11: D1.1 (K), E1.54, IC2.1 (A11), IC25.5 (2A), IC3.5 (2A), IC5.23 (A11)
- new net A12: D4.1 (K), E1.29, IC2.2 (A12), IC25.2 (1A), IC3.2 (1A), IC5.2 (A12)
- new net A13: D5.1 (K), E1.2, IC2.3 (A13), IC25.14 (4A), IC3.14 (4A), IC5.26 (A13)
- new net A14: D7.1 (K), E1.28, IC1.36 (A14), IC2.4 (A14), J3.1 (Pin_1), J4.1 (Pin_1)
- new net A15: D8.1 (K), E1.1, IC1.37 (A15), IC2.5 (A15), IC24.10
- new net A2: E1.37, IC2.32 (A2), IC26.13 (4B), IC4.13 (4B), IC5.8 (A2)
- new net A3: E1.38, IC2.33 (A3), IC25.10 (3B), IC3.10 (3B), IC5.7 (A3)
- new net A4: E1.50, IC2.34 (A4), IC25.6 (2B), IC3.6 (2B), IC5.6 (A4)
- new net A5: E1.49, IC2.35 (A5), IC25.3 (1B), IC3.3 (1B), IC5.5 (A5)
- new net A6: E1.48, IC2.36 (A6), IC25.13 (4B), IC3.13 (4B), IC5.4 (A6)
- new net A7: E1.47, IC2.37 (A7), IC26.5 (2A), IC4.5 (2A), IC5.3 (A7)
- new net A8: D6.1 (K), E1.25, IC2.38 (A0), IC26.2 (1A), IC4.2 (1A), IC5.25 (A8)
- new net A9: D3.1 (K), E1.53, IC2.39 (A9), IC26.14 (4A), IC4.14 (4A), IC5.24 (A9)
- new net D0: E1.5, IC15.14 (G), IC15.2 (D), IC2.14 (D0), IC5.11 (D0), R1.1, R9.2
- new net D1: E1.6, IC16.14 (G), IC16.2 (D), IC2.15 (D1), IC5.12 (D1), R10.2, R2.1
- new net D2: E1.7, IC17.14 (G), IC17.2 (D), IC2.12 (D2), IC5.13 (D2), R11.2, R3.1
- new net D3: E1.10, IC18.14 (G), IC18.2 (D), IC2.8 (D3), IC5.15 (D3), R12.2, R4.1
- new net D4: E1.11, IC19.14 (G), IC19.2 (D), IC2.7 (D4), IC5.16 (D4), R13.2, R5.1
- new net D5: E1.9, IC2.9 (D5), IC20.14 (G), IC20.2 (D), IC5.17 (D5), R14.2, R6.1
- new net D6: E1.8, IC2.10 (D6), IC21.14 (G), IC21.2 (D), IC5.18 (D6), R15.2, R7.1
- new net D7: E1.3, IC2.13 (D7), IC22.14 (G), IC22.2 (D), IC5.19 (D7), R16.2, R8.1
- new net LA0: IC1.5 (A0), IC10.7 (A1), IC11.7 (A1), IC12.7 (A1), IC13.7 (A1), IC6.7 (A1), IC7.7 (A1), IC8.7 (A1), IC9.7 (A1), R17.2
- new net LA1: IC1.6 (A1), IC10.11 (A4), IC11.11 (A4), IC12.11 (A4), IC13.11 (A4), IC6.11 (A4), IC7.11 (A4), IC8.11 (A4), IC9.11 (A4), R18.2
- new net LA2: IC1.7 (A2), IC10.5 (A0), IC11.5 (A0), IC12.5 (A0), IC13.5 (A0), IC6.5 (A0), IC7.5 (A0), IC8.5 (A0), IC9.5 (A0), R19.2
- new net LA3: IC1.8 (A3), IC10.13 (A6), IC11.13 (A6), IC12.13 (A6), IC13.13 (A6), IC6.13 (A6), IC7.13 (A6), IC8.13 (A6), IC9.13 (A6), R20.2
- new net LA4: IC1.9 (A4), IC10.12 (A3), IC11.12 (A3), IC12.12 (A3), IC13.12 (A3), IC6.12 (A3), IC7.12 (A3), IC8.12 (A3), IC9.12 (A3), R21.2
- new net LA5: IC1.10 (A5), IC10.10 (A5), IC11.10 (A5), IC12.10 (A5), IC13.10 (A5), IC6.10 (A5), IC7.10 (A5), IC8.10 (A5), IC9.10 (A5), R22.2
- new net LA6: IC1.11 (A6), IC10.6 (A2), IC11.6 (A2), IC12.6 (A2), IC13.6 (A2), IC6.6 (A2), IC7.6 (A2), IC8.6 (A2), IC9.6 (A2), R23.2
- new net LDRAM_WE: IC1.4 (DRAMWE), IC10.3 (~{WRITE}), IC11.3 (~{WRITE}), IC12.3 (~{WRITE}), IC13.3 (~{WRITE}), IC6.3 (~{WRITE}), IC7.3 (~{WRITE}), IC8.3 (~{WRITE}), IC9.3 (~{WRITE})
- new net U: C69.2, E1.44, IC1.15 (u), R56.1
- new net UA0: IC15.5 (A0), IC16.5 (A0), IC17.5 (A0), IC18.5 (A0), IC19.5 (A0), IC20.5 (A0), IC21.5 (A0), IC22.5 (A0), IC26.7 (2Y)
- new net UA1: IC15.7 (A1), IC16.7 (A1), IC17.7 (A1), IC18.7 (A1), IC19.7 (A1), IC20.7 (A1), IC21.7 (A1), IC22.7 (A1), IC26.12 (4Y)
- new net UA2: IC15.6 (A2), IC16.6 (A2), IC17.6 (A2), IC18.6 (A2), IC19.6 (A2), IC20.6 (A2), IC21.6 (A2), IC22.6 (A2), IC26.4 (1Y)
- new net UA3: IC15.12 (A3), IC16.12 (A3), IC17.12 (A3), IC18.12 (A3), IC19.12 (A3), IC20.12 (A3), IC21.12 (A3), IC22.12 (A3), IC25.9 (3Y)
- new net UA4: IC15.11 (A4), IC16.11 (A4), IC17.11 (A4), IC18.11 (A4), IC19.11 (A4), IC20.11 (A4), IC21.11 (A4), IC22.11 (A4), IC25.7 (2Y)
- new net UA5: IC15.10 (A5), IC16.10 (A5), IC17.10 (A5), IC18.10 (A5), IC19.10 (A5), IC20.10 (A5), IC21.10 (A5), IC22.10 (A5), IC25.4 (1Y)
- new net UA6: IC15.13 (A6), IC16.13 (A6), IC17.13 (A6), IC18.13 (A6), IC19.13 (A6), IC20.13 (A6), IC21.13 (A6), IC22.13 (A6), IC25.12 (4Y)
- new net UA7: IC15.9 (A7), IC16.9 (A7), IC17.9 (A7), IC18.9 (A7), IC19.9 (A7), IC20.9 (A7), IC21.9 (A7), IC22.9 (A7), IC26.9 (3Y)
- new net V: C71.2, E1.43, IC1.16 (v), R63.1
- new net VIDEO: E1.41, R53.2, TR2.3 (E), TV1.2 (1P)
- new net Y: C68.2, C70.2, E1.42, IC1.17 (h), R47.2, R48.2
- new net _BUSACK: E1.52, IC2.23 (~{BUSACK})
- new net _BUS_REQ: E1.45, IC2.25 (~{BUSRQ}), R30.2
- new net _CK: C67.1, E1.34, IC1.32 (_CPU), R24.2, R73.2
- new net _HALT: E1.14, IC2.18 (~{HALT})
- new net _INT: E1.12, IC2.16 (~{INT}), R26.1
- new net _IO_REQ: E1.16, IC2.20 (~{IORQ}), R27.1
- new net _IO_RQULA: E1.39, IC1.33 (_IOREQ), R27.2, TR6.3 (E)
- new net _LCAS: IC1.1 (_CAS), IC10.15 (~{CAS}), IC11.15 (~{CAS}), IC12.15 (~{CAS}), IC13.15 (~{CAS}), IC6.15 (~{CAS}), IC7.15 (~{CAS}), IC8.15 (~{CAS}), IC9.15 (~{CAS})
- new net _LRAS: IC1.35 (_RAS), IC10.4 (~{RAS}), IC11.4 (~{RAS}), IC12.4 (~{RAS}), IC13.4 (~{RAS}), IC6.4 (~{RAS}), IC7.4 (~{RAS}), IC8.4 (~{RAS}), IC9.4 (~{RAS}), R32.2
- new net _M1: E1.23, IC2.27 (~{M1})
- new net _M_REQ: E1.15, IC1.38 (_MREQ), IC2.19 (~{MREQ}), IC23.1, IC23.2, J10.1 (Pin_1)
- new net _NMI: E1.13, IC2.17 (~{NMI}), R28.2
- new net _RD: E1.17, IC1.3 (_R0), IC2.21 (~{RD}), IC24.4, IC5.22 (OE0L)
- new net _RESET: C27.1, E1.46, IC2.26 (~{RESET}), R31.2
- new net _RFSH: E1.24, IC2.28 (~{RFSH})
- new net _ROMCS: E1.51, J9.1 (Pin_1), R33.1
- new net _UCAS: IC15.15 (~{CAS}), IC16.15 (~{CAS}), IC17.15 (~{CAS}), IC18.15 (~{CAS}), IC19.15 (~{CAS}), IC20.15 (~{CAS}), IC21.15 (~{CAS}), IC22.15 (~{CAS}), IC23.6
- new net _URAS: IC15.4 (~{RAS}), IC16.4 (~{RAS}), IC17.4 (~{RAS}), IC18.4 (~{RAS}), IC19.4 (~{RAS}), IC20.4 (~{RAS}), IC21.4 (~{RAS}), IC22.4 (~{RAS}), IC23.3, IC23.4, R71.1
- new net _UWRITE: IC15.3 (~{WRITE}), IC16.3 (~{WRITE}), IC17.3 (~{WRITE}), IC18.3 (~{WRITE}), IC19.3 (~{WRITE}), IC20.3 (~{WRITE}), IC21.3 (~{WRITE}), IC22.3 (~{WRITE}), IC23.11, IC24.5
- new net _WAIT: E1.20, IC2.24 (~{WAIT}), R29.2
- new net _WR: E1.18, IC1.2 (_WR), IC2.22 (~{WR}), IC23.12, IC23.13
- no-connect marks 0 -> 2
Other:
- company: (none) -> Submeson Brain Corperation
- title: (none) -> ZX Spectrum 48K

Commit message: Added Schematic PDF
Parts:
- removed R79: 2k2, symbol Device:R
- R10, R11, R12, R13, R14, R15, R16, R9: value 8k2 -> 8K2
- R48: value 4K7 -> 2K2
- R50: value 8K2 -> 4K7
- TR5: value ZTX313 -> ZTX213
- renumbered D18 to D12, D19 to D16
Connections:
- net +5V: now also D12.2 (A)
Other:
- moved on the sheet: D12
Changed lines of the file:
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@@
 	(wire
 		(pts
-			(xy 124.46 499.11) (xy 116.84 499.11)
+			(xy 132.08 499.11) (xy 116.84 499.11)
 		)
 		(stroke
@@
 	(wire
 		(pts
-			(xy 152.4 499.11) (xy 151.13 499.11)
-		)
-		(stroke
-			(width 0)
-			(type default)
-		)
-	)
-	(wire
-		(pts
 			(xy 373.38 424.18) (xy 373.38 443.23)
 		)
@@
 	(wire
 		(pts
-			(xy 132.08 499.11) (xy 143.51 499.11)
+			(xy 139.7 499.11) (xy 152.4 499.11)
 		)
 		(stroke
@@
 			)
 		)
-		(property "Value" "8k2"
+		(property "Value" "8K2"
 			(at 368.3 426.72 90)
 			(effects
@@
 			)
 		)
-		(property "Value" "8k2"
+		(property "Value" "8K2"
 			(at 372.11 426.72 90)
 			(effects
@@
 			)
 		)
-		(property "Value" "8k2"
+		(property "Value" "8K2"
 			(at 375.92 426.72 90)
 			(effects
@@
 			)
 		)
-		(property "Value" "8k2"
+		(property "Value" "8K2"
 			(at 379.73 426.72 90)
 			(effects
@@
 			)
 		)
-		(property "Value" "8k2"
+		(property "Value" "8K2"
 			(at 383.54 426.72 90)
 			(effects
@@
 			)
 		)
-		(property "Value" "8k2"
+		(property "Value" "8K2"
 			(at 387.35 426.72 90)
 			(effects
@@
 			)
 		)
-		(property "Value" "8k2"
+		(property "Value" "8K2"
 			(at 391.16 426.72 90)
 			(effects
@@
 			)
 		)
-		(property "Value" "8k2"
+		(property "Value" "8K2"
 			(at 394.97 426.72 90)
 			(effects
@@
 	(symbol
 		(lib_id "Diode:1N4148")
-		(at 128.27 499.11 0)
+		(at 135.89 499.11 0)
 		(unit 1)
 		(exclude_from_sim no)
@@
 		(on_board yes)
 		(dnp no)
-		(property "Reference" "D18"
-			(at 130.81 501.65 0)
+		(property "Reference" "D12"
+			(at 138.43 501.65 0)
 			(effects
 				(font
@@
 		)
 		(property "Value" "1N4148"
-			(at 127.127 501.142 90)
+			(at 134.747 501.142 90)
 			(effects
 				(font
@@
 		)
 		(property "Footprint" ""
-			(at 128.27 503.555 0)
+			(at 135.89 503.555 0)
 			(effects
 				(font
@@
 		)
 		(property "Datasheet" "https://assets.nexperia.com/documents/data-sheet/1N4148_1N4448.pdf"
-			(at 128.27 499.11 0)
+			(at 135.89 499.11 0)
 			(effects
 				(font
@@
 		)
 		(property "Description" ""
-			(at 128.27 499.11 0)
+			(at 135.89 499.11 0)
 			(effects
 				(font
@@
 			(project ""
 				(path "/07f22ea6-4813-487d-9e01-b5b6de3af68a"
-					(reference "D18")
+					(reference "D12")
 					(unit 1)
 				)
@@
 		(on_board yes)
 		(dnp no)
-		(property "Reference" "D19"
+		(property "Reference" "D16"
 			(at 154.432 490.3216 90)
 			(effects
@@
 			(project ""
 				(path "/07f22ea6-4813-487d-9e01-b5b6de3af68a"
-					(reference "D19")
+					(reference "D16")
 					(unit 1)
 				)
@@
 	)
 	(symbol
-		(lib_id "Device:R")
-		(at 147.32 499.11 90)
-		(unit 1)
-		(exclude_from_sim no)
-		(in_bom yes)
-		(on_board yes)
-		(dnp no)
-		(property "Reference" "R79"
-			(at 146.05 496.57 90)
-			(effects
-				(font
-					(size 1.27 1.27)
-				)
-			)
-		)
-		(property "Value" "2k2"
-			(at 146.05 501.65 90)
-			(effects
-				(font
-					(size 1.27 1.27)
-				)
-			)
-		)
-		(property "Footprint" ""
-			(at 147.32 500.888 90)
-			(effects
-				(font
-					(size 1.27 1.27)
-				)
-				(hide yes)
-			)
-		)
-		(property "Datasheet" "~"
-			(at 147.32 499.11 0)
-			(effects
-				(font
-					(size 1.27 1.27)
-				)
-				(hide yes)
-			)
-		)
-		(property "Description" ""
-			(at 147.32 499.11 0)
-			(effects
-				(font
-					(size 1.27 1.27)
-				)
-				(hide yes)
-			)
-		)
-		(pin "1"
-		)
-		(pin "2"
-		)
-		(instances
-			(project ""
-				(path "/07f22ea6-4813-487d-9e01-b5b6de3af68a"
-					(reference "R79")
-					(unit 1)
-				)
-			)
-		)
-	)
-	(symbol
 		(lib_id "Issue 4-rescue:GND-power")
 		(at 707.39 226.06 90)
@@
 			)
 		)
-		(property "Value" "4K7"
+		(property "Value" "2K2"
 			(at 116.84 255.27 90)
 			(effects
@@
 			)
 		)
-		(property "Value" "8K2"
+		(property "Value" "4K7"
 			(at 104.14 247.65 90)
 			(effects
@@
 			)
 		)
-		(property "Value" "ZTX313"
+		(property "Value" "ZTX213"
 			(at 38.3286 425.323 0)
 			(effects

Commit message: Updated schematic re produced schematic pdf
Parts:
- added R25: 180, symbol Device:R
- added R54: 100K, symbol Device:R
- added R55: 56, symbol Device:R
- D16: value DZY88 -> 5V1
- J3: value TI -> OKI
- X2: value 4.43Mhz -> 4.433619Mhz
Connections:
- net +5V: now also C47.1, C47.2, R25.2, R54.1, R54.2; no longer D16.2 (A), IC2.6 (~{CLK}), TR3.1 (C)
- net -12V: now also D15.2 (A); no longer C47.1
- net at C46.2, D11.2 (A): now also R55.1; no longer D12.1 (K)
- new net: IC2.6 (~{CLK}), R25.1, TR3.1 (C)
- new net: D12.1 (K), D16.2 (A), R55.2
Other:
- moved on the sheet: C34, C43, C44, C45, C46, C47, C49, C50, C66, C74, C77, D11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
