File: src/issue3b.kicad_sch (KiCad schematic)
At the start: 199 parts, among them IC1 ULA, IC10 4116, IC11 4116, IC12 4116, IC13 4116, IC14 LM1889, IC15 4532, IC16 4532, IC17 4532, IC18 4532, IC19 4532, IC2 Z80, IC20 4532, IC21 4532, IC22 4532, IC23 74LS32, IC24 74LS00, IC25 74LS157, IC26 74LS157, IC3 74LS157, IC4 74LS157, IC5 ROM, IC6 4116, IC7 4116, IC8 4116, IC9 4116, J1 OKI, J10 UR3, J11 UR4, J2 TI, J3 OKI, J4 TI, J7 Barrel_Jack_MountingPin, J8 UR1, J9 UR2, T1 Coil, X1 14Mhz, X2 4.433619Mhz

Commit message: added some new footprints
Parts:
- removed C47: 22uF, Capacitor_THT:CP_Axial_L11.0mm_D6.0mm_P18.00mm_Horizontal, symbol Issue 4-rescue:CP_Small-Device
- removed D12: 1N4148, symbol Diode:1N4148
- removed J1, J3: OKI, Connector_PinHeader_2.54mm:PinHeader_1x03_P2.54mm_Vertical, symbol Connector_Generic:Conn_01x03
- removed J10: UR3, Connector_PinHeader_2.54mm:PinHeader_1x01_P2.54mm_Vertical, symbol Connector_Generic:Conn_01x01
- removed J11: UR4, Connector_PinHeader_2.54mm:PinHeader_1x01_P2.54mm_Vertical, symbol Connector_Generic:Conn_01x01
- removed J2, J4: TI, Connector_PinHeader_2.54mm:PinHeader_1x03_P2.54mm_Vertical, symbol Connector_Generic:Conn_01x03
- removed J8: UR1, Connector_PinHeader_2.54mm:PinHeader_1x01_P2.54mm_Vertical, symbol Connector_Generic:Conn_01x01
- removed J9: UR2, Connector_PinHeader_2.54mm:PinHeader_1x01_P2.54mm_Vertical, symbol Connector_Generic:Conn_01x01
- added C47: 22uF, symbol ZXSpectrumIssue3B:Capacitor Electrolytic
- added C63: 47pF, spectrum3b:Passive, symbol Device:C_Small
- added D12: 1N4148, symbol ZXSpectrumIssue3B:1N4148
- added unit 1 of IC24
- added unit 4 of IC24
- added JROM1: JROM, symbol Connector_Generic:Conn_02x02_Odd_Even
- added OKI-H1: OKI-H, symbol Connector_Generic:Conn_01x02
- added OKI-L1: OKI-L, symbol Connector_Generic:Conn_01x02
- added OKI1: OKI, symbol Connector_Generic:Conn_01x02
- added TI-3: TI-3, symbol Connector_Generic:Conn_01x02
- added TI-4: TI-4, symbol Connector_Generic:Conn_01x02
- added TI1: TI, symbol Connector_Generic:Conn_01x02
- C1, C2, C26, C29, C3, C30, C31, C32, C33, C35, C37, C38, C39, C4, C40, C41, C42, C43, C48, C49, C5, C52, C53, C55, C56, C57, C58, C59, C6, C60, C61, C62, C64, C66, C67, C68, C69, C7, C70, C71, C72, C73, C75, C76, C77, C8, R1, R17, R18, R19, R2, R20, R21, R22, R23, R25, R26, R27, R28, R29, R3, R30, R31, R32, R33, R35, R36, R37, R4, R42, R43, R44, R45, R46, R47, R48, R49, R5, R50, R51, R52, R53, R54, R55, R56, R6, R61, R62, R63, R64, R65, R66, R67, R68, R69, R7, R70, R71, R72, R74, R75, R76, R77, R78, R8: footprint (none) -> spectrum3b:Passive
- C25, C27, C28, C34, C46, C50, C65, C74: footprint Capacitor_THT:CP_Axial_L11.0mm_D6.0mm_P18.00mm_Horizontal -> (none); symbol Issue 4-rescue:CP_Small-Device -> ZXSpectrumIssue3B:Capacitor Electrolytic
- C44, C45: footprint Capacitor_THT:CP_Axial_L11.0mm_D6.0mm_P18.00mm_Horizontal -> spectrum3b:Passive; symbol Issue 4-rescue:CP_Small-Device -> ZXSpectrumIssue3B:Capacitor Electrolytic
- D1, D11, D13, D15, D2, D3, D4, D5, D6, D7, D8, D9: symbol Diode:1N4148 -> ZXSpectrumIssue3B:1N4148
- D16: value 5V1 -> DZY88; footprint Diode_THT:D_DO-35_SOD27_P7.62mm_Horizontal -> (none)
- E1: symbol Issue-4-rescue:Edge_Connector-spectrum -> ZXSpectrumIssue3B:Edge_Connector-spectrum
- Ear0, Mic0: symbol Connector:Barrel_Jack -> ZXSpectrumIssue3B:Barrel_Jack
- IC1: footprint Package_DIP:DIP-40_W15.24mm_Socket -> (none); symbol Issue-4-rescue:ULA-spectrum -> ZXSpectrumIssue3B:ULA-spectrum
- IC10, IC11, IC12, IC13, IC6, IC7, IC8, IC9: footprint Package_DIP:DIP-16_W7.62mm_Socket -> (none); symbol Issue-4-rescue:4116-spectrum -> ZXSpectrumIssue3B:4116-spectrum
- IC14: footprint Package_DIP:DIP-18_W7.62mm_Socket -> (none); symbol Issue-4-rescue:LM1809-spectrum -> ZXSpectrumIssue3B:LM1809-spectrum
- IC15, IC16, IC17, IC18, IC19, IC20, IC21, IC22: footprint Package_DIP:DIP-16_W7.62mm_Socket -> (none); symbol Issue-4-rescue:4532-spectrum -> ZXSpectrumIssue3B:4532-spectrum
- IC2: footprint Package_DIP:DIP-40_W15.24mm_Socket -> (none); symbol Issue-4-rescue:Z80-spectrum -> ZXSpectrumIssue3B:Z80-spectrum
- IC23, IC24: footprint Package_DIP:DIP-14_W7.62mm_Socket -> (none)
- IC25, IC26: footprint Package_DIP:DIP-16_W7.62mm_Socket -> (none); symbol Issue-4-rescue:74LS157-spectrum -> ZXSpectrumIssue3B:74LS157-spectrum
- IC3: value 74LS157 -> LS157; footprint Package_DIP:DIP-16_W7.62mm_Socket -> (none); symbol Issue-4-rescue:LS157-spectrum -> ZXSpectrumIssue3B:LS157-spectrum
- IC4: value 74LS157 -> LS157; footprint Package_DIP:DIP-16_W7.62mm_Socket -> (none); symbol Issue-4-rescue:LS157-A-spectrum -> ZXSpectrumIssue3B:LS157-A-spectrum
- IC5: footprint Package_DIP:DIP-28_W15.24mm_Socket -> (none); symbol Issue-4-rescue:ROM-spectrum -> ZXSpectrumIssue3B:ROM-spectrum
- J7: symbol Connector:Barrel_Jack_MountingPin -> ZXSpectrumIssue3B:Barrel_Jack_MountingPin
- KB1: footprint Connector_PinSocket_2.54mm:PinSocket_1x05_P2.54mm_Vertical -> (none)
- KB2: footprint Connector_PinSocket_2.54mm:PinSocket_1x08_P2.54mm_Vertical -> (none)
- LS1: footprint (none) -> spectrum3b:Speaker
- R10, R11, R12, R13, R14, R15, R16, R9: value 8K2 -> 8k2; footprint (none) -> spectrum3b:Passive
- R24, R73: value 1K -> 1k; footprint (none) -> spectrum3b:Passive
- R34: value 15 1W -> 15; footprint Resistor_THT:R_Axial_Power_L20.0mm_W6.4mm_P22.40mm -> (none)
- R58: value 1K 2% -> 1K; footprint (none) -> spectrum3b:Passive
- R59: value 1K8 2% -> 1K8; footprint (none) -> spectrum3b:Passive
- R60: value 68 -> 68R; footprint (none) -> spectrum3b:Passive
- REG1: symbol Regulator_Linear:L7805 -> ZXSpectrumIssue3B:L7805
- T1: footprint (none) -> spectrum3b:Coil
- TR1, TR2, TR3, TR4, TR6, TR7: footprint Package_TO_SOT_THT:TO-92Flat -> (none); symbol Transistor_BJT:BC547 -> ZXSpectrumIssue3B:Transistor NPN
- TR5: footprint Package_TO_SOT_THT:TO-92Flat -> (none); symbol Device:Q_PNP_CBE -> ZXSpectrumIssue3B:Transistor_PNP
- TR8, TR9: footprint Package_TO_SOT_THT:TO-92_Inline -> (none); symbol Transistor_BJT:BC547 -> ZXSpectrumIssue3B:Transistor NPN
- TV1: footprint (none) -> spectrum3b:Modulator; symbol Issue-4-rescue:Modulator -> ZXSpectrumIssue3B:Modulator
- X1: footprint Crystal:Crystal_HC18-U_Vertical -> spectrum3b:X1
- X2: value 4.433619Mhz -> 4.43Mhz; footprint Crystal:Crystal_HC18-U_Horizontal -> spectrum3b:X2
Connections:
- net +5V: now also R25.1, IC24.1, IC24.12, IC24.13, IC24.2, OKI-H1.1 (Pin_1), TI-4.1 (Pin_1); no longer C1.1, C1.2, C2.1, C2.2, C25.2, C26.2, C27.2, C28.2, C29.1, C3.1, C3.2, C30.1, C33.1, C34.2, C35.1, C37.2, C4.1, C4.2, C40.2, C41.2, C42.2, C43.1, C44.2, C45.2, C48.1, C49.1, C5.2, C50.2, C55.1, C56.1, C57.1, C58.1, C59.1, C6.2, C60.1, C61.1, C62.1, C64.2, C66.1, C7.2, C72.2, C73.1, C75.1, C76.1, C77.1, C8.2, D11.1 (K), D13.2 (A), D16.1 (K), E1.19, E1.32, E1.33, E1.40, Ear0.1, IC1.40 (GND), IC10.1 (VBB), IC10.16 (VSS), IC11.1 (VBB), IC11.16 (VSS), IC12.1 (VBB), IC12.16 (VSS), IC13.1 (VBB), IC13.16 (VSS), IC14.5 (GROUND), IC15.1 (NC), IC15.16 (VSS), IC16.1 (NC), IC16.16 (VSS), IC17.1 (NC), IC17.16 (VSS), IC18.1 (NC), IC18.16 (VSS), IC19.1 (NC), IC19.16 (VSS), IC2.29 (GND), IC20.1 (NC), IC20.16 (VSS), IC21.1 (NC), IC21.16 (VSS), IC22.1 (NC), IC22.16 (VSS), IC23.7 (GND), IC23.9, IC24.7 (GND), IC25.15 (STROBE), IC25.8 (GND), IC26.15 (STROBE), IC26.8 (GND), IC3.15 (STROBE), IC3.8 (GND), IC4.15 (STROBE), IC4.8 (GND), IC5.14 (Vss), IC6.1 (VBB), IC6.16 (VSS), IC7.1 (VBB), IC7.16 (VSS), IC8.1 (VBB), IC8.16 (VSS), IC9.1 (VBB), IC9.16 (VSS), J7.1, LS1.1, Mic0.1, R25.2, R37.2, R43.1, R46.1, R47.1, R50.1, R52.1, R53.1, R54.1, R54.2, R56.2, R58.2, R63.2, R71.2, REG1.2 (GND), TR3.3 (E), TR4.3 (E), TV1.3 (GND)
- net A14: now also OKI1.2 (Pin_2), TI1.2 (Pin_2)
- net _M_REQ: now also JROM1.2 (Pin_2)
- net _ROMCS: now also JROM1.3 (Pin_3)
- net at IC2.6 (~{CLK}), TR3.1 (C): now also R25.2; no longer R25.1
- net at IC5.20 (CS): now also JROM1.1 (Pin_1)
- net at IC5.27 (OE1L): now also JROM1.4 (Pin_4)
- net at IC26.10 (3B): now also OKI1.1 (Pin_1), TI-3.2 (Pin_2), TI-4.2 (Pin_2)
- net at D16.2 (A), R55.2: now also D12.1 (K)
- net at IC26.11 (3A): now also OKI-H1.2 (Pin_2), OKI-L1.2 (Pin_2), TI1.1 (Pin_1)
- net -12V renamed -12VAC
- new net: C63.1, IC23.9, R71.2
- new net -5V: C1.1, C2.1, C3.1, C4.1, C47.2, D12.2 (A), E1.19, IC10.1 (VBB), IC11.1 (VBB), IC12.1 (VBB), IC13.1 (VBB), IC6.1 (VBB), IC7.1 (VBB), IC8.1 (VBB), IC9.1 (VBB), R54.1
- new net GND: C1.2, C2.2, C25.2, C26.2, C27.2, C28.2, C29.1, C3.2, C30.1, C33.1, C34.2, C35.1, C37.2, C4.2, C40.2, C41.2, C42.2, C43.1, C44.2, C45.2, C47.1, C48.1, C49.1, C5.2, C50.2, C55.1, C56.1, C57.1, C58.1, C59.1, C6.2, C60.1, C61.1, C62.1, C63.2, C64.2, C66.1, C7.2, C72.2, C73.1, C75.1, C76.1, C77.1, C8.2, D11.1 (K), D13.2 (A), D16.1 (K), E1.32, E1.33, E1.40, Ear0.1, IC1.40 (GND), IC10.16 (VSS), IC11.16 (VSS), IC12.16 (VSS), IC13.16 (VSS), IC14.5 (GROUND), IC15.1 (NC), IC15.16 (VSS), IC16.1 (NC), IC16.16 (VSS), IC17.1 (NC), IC17.16 (VSS), IC18.1 (NC), IC18.16 (VSS), IC19.1 (NC), IC19.16 (VSS), IC2.29 (GND), IC20.1 (NC), IC20.16 (VSS), IC21.1 (NC), IC21.16 (VSS), IC22.1 (NC), IC22.16 (VSS), IC23.7 (GND), IC24.7 (GND), IC25.15 (STROBE), IC25.8 (GND), IC26.15 (STROBE), IC26.8 (GND), IC3.15 (STROBE), IC3.8 (GND), IC4.15 (STROBE), IC4.8 (GND), IC5.14 (Vss), IC6.16 (VSS), IC7.16 (VSS), IC8.16 (VSS), IC9.16 (VSS), J7.1, LS1.1, Mic0.1, OKI-L1.1 (Pin_1), R37.2, R43.1, R46.1, R47.1, R50.1, R52.1, R53.1, R54.2, R56.2, R58.2, R63.2, REG1.2 (GND), TI-3.1 (Pin_1), TR3.3 (E), TR4.3 (E), TV1.3 (GND)
- no-connect marks 2 -> 4
Other:
- title: ZX Spectrum 48K -> ZX Spectrum
- moved on the sheet: C34, C43, C44, C45, C46, C49, C50, C55, C56, C57, C58, C59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
