File: src/issue3b.kicad_pcb (KiCad board)
At the start: 2 copper layers, 213.1 x 129 mm, 0 parts

Commit message: added some new footprints
Parts:
- added C1: 47nF, spectrum3b:Passive, F.Cu at (56.3, 121.9)
- added C2: 47nF, spectrum3b:Passive, F.Cu at (-125.6, -23.3)
- added C26: 47nF, spectrum3b:Passive, F.Cu at (-125.6, 5.02)
- added C29: 47nF, spectrum3b:Passive, F.Cu at (-125.6, 9.07)
- added C3: 47nF, spectrum3b:Passive, F.Cu at (-125.6, -19.3)
- added C30: 47nF, spectrum3b:Passive, F.Cu at (-125.6, 13.1)
- added C31: 100nF, spectrum3b:Passive, F.Cu at (-125.6, 17.2)
- added C32: 100nF, spectrum3b:Passive, F.Cu at (-125.6, 21.2)
- added C33: 47nF, spectrum3b:Passive, F.Cu at (-125.6, 25.3)
- added C35: 10nF, spectrum3b:Passive, F.Cu at (-125.6, 29.3)
- added C37: 33pF, spectrum3b:Passive, F.Cu at (-125.6, 33.4)
- added C38: 33pF, spectrum3b:Passive, F.Cu at (-125.6, 37.4)
- added C39: 10nF, spectrum3b:Passive, F.Cu at (-125.6, 41.4)
- added C4: 47nF, spectrum3b:Passive, F.Cu at (-125.6, -15.2)
- added C40: 47nF, spectrum3b:Passive, F.Cu at (-125.6, 45.5)
- added C41: 47nF, spectrum3b:Passive, F.Cu at (-125.6, 49.5)
- added C42: 47nF, spectrum3b:Passive, F.Cu at (-125.6, 53.6)
- added C43: 100nF, spectrum3b:Passive, F.Cu at (-110.1, -27.4)
- added C44: 100uF, spectrum3b:Passive, F.Cu at (-110.1, -23.3)
- added C45: 100uF, spectrum3b:Passive, F.Cu at (-110.1, -19.3)
- added C48: 47nF, spectrum3b:Passive, F.Cu at (-110.1, -15.2)
- added C49: 560pF, spectrum3b:Passive, F.Cu at (-110.1, -11.2)
- added C5: 47nF, spectrum3b:Passive, F.Cu at (-125.6, -11.2)
- added C52: 150pF, spectrum3b:Passive, F.Cu at (-110.1, -7.13)
- added C53: 150pF, spectrum3b:Passive, F.Cu at (-110.1, -3.08)
- added C55: 47nF, spectrum3b:Passive, F.Cu at (-110.1, 0.97)
- added C56: 47nF, spectrum3b:Passive, F.Cu at (-110.1, 5.02)
- added C57: 47nF, spectrum3b:Passive, F.Cu at (-110.1, 9.07)
- added C58: 47nF, spectrum3b:Passive, F.Cu at (-110.1, 13.1)
- added C59: 47nF, spectrum3b:Passive, F.Cu at (-110.1, 17.2)
- added C6: 47nF, spectrum3b:Passive, F.Cu at (-125.6, -7.13)
- added C60: 47nF, spectrum3b:Passive, F.Cu at (-110.1, 21.2)
- added C61: 47nF, spectrum3b:Passive, F.Cu at (-110.1, 25.3)
- added C62: 47nF, spectrum3b:Passive, F.Cu at (-110.1, 29.3)
- added C63: 47pF, spectrum3b:Passive, F.Cu at (-110.1, 33.4)
- added C64: 100pF, spectrum3b:Passive, F.Cu at (-110.1, 37.4)
- added C66: 47nF, spectrum3b:Passive, F.Cu at (-110.1, 41.4)
- added C67: 100pF, spectrum3b:Passive, F.Cu at (-110.1, 45.5)
- added C68: 100nF, spectrum3b:Passive, F.Cu at (-110.1, 49.5)
- added C69: 100nF, spectrum3b:Passive, F.Cu at (-110.1, 53.6)
- added C7: 47nF, spectrum3b:Passive, F.Cu at (-125.6, -3.08)
- added C70: 100nF, spectrum3b:Passive, F.Cu at (-94.6, -27.4)
- added C71: 100nF, spectrum3b:Passive, F.Cu at (-94.6, -23.3)
- added C72: 16pF, spectrum3b:Passive, F.Cu at (-94.6, -19.3)
- added C73: 16pF, spectrum3b:Passive, F.Cu at (-94.6, -15.2)
- added C75: 100nF, spectrum3b:Passive, F.Cu at (-94.6, -11.2)
- added C76: 47nF, spectrum3b:Passive, F.Cu at (-94.6, -7.13)
- added C77: 100nF, spectrum3b:Passive, F.Cu at (-94.6, -3.08)
- added C8: 47nF, spectrum3b:Passive, F.Cu at (-125.6, 0.97)
- added LS1: Speaker, spectrum3b:Speaker, F.Cu at (233.9, 141.2)
- added R1: 470, spectrum3b:Passive, F.Cu at (-94.6, 0.97)
- added R10: 8k2, spectrum3b:Passive, F.Cu at (-94.6, 37.4)
- added R11: 8k2, spectrum3b:Passive, F.Cu at (-94.6, 41.4)
- added R12: 8k2, spectrum3b:Passive, F.Cu at (-94.6, 45.5)
- added R13: 8k2, spectrum3b:Passive, F.Cu at (-94.6, 49.5)
- added R14: 8k2, spectrum3b:Passive, F.Cu at (-94.6, 53.6)
- added R15: 8k2, spectrum3b:Passive, F.Cu at (-79.0, -27.4)
- added R16: 8k2, spectrum3b:Passive, F.Cu at (-79.0, -23.3)
- added R17: 330, spectrum3b:Passive, F.Cu at (-79.0, -19.3)
- added R18: 330, spectrum3b:Passive, F.Cu at (-79.0, -15.2)
- added R19: 330, spectrum3b:Passive, F.Cu at (-79.0, -11.2)
- added R2: 470, spectrum3b:Passive, F.Cu at (-94.6, 5.02)
- added R20: 330, spectrum3b:Passive, F.Cu at (-79.0, -7.13)
- added R21: 330, spectrum3b:Passive, F.Cu at (-79.0, -3.08)
- added R22: 330, spectrum3b:Passive, F.Cu at (-79.0, 0.97)
- added R23: 330, spectrum3b:Passive, F.Cu at (-79.0, 5.02)
- added R24: 1k, spectrum3b:Passive, F.Cu at (-79.0, 9.07)
- added R25: 180, spectrum3b:Passive, F.Cu at (-79.0, 13.1)
- added R26: 470, spectrum3b:Passive, F.Cu at (-79.0, 17.2)
- added R27: 470, spectrum3b:Passive, F.Cu at (-79.0, 21.2)
- added R28: 10K, spectrum3b:Passive, F.Cu at (-79.0, 25.3)
- added R29: 10K, spectrum3b:Passive, F.Cu at (-79.0, 29.3)
- added R3: 470, spectrum3b:Passive, F.Cu at (-94.6, 9.07)
- added R30: 10K, spectrum3b:Passive, F.Cu at (-79.0, 33.4)
- added R31: 220K, spectrum3b:Passive, F.Cu at (-79.0, 37.4)
- added R32: 100, spectrum3b:Passive, F.Cu at (-79.0, 41.4)
- added R33: 680, spectrum3b:Passive, F.Cu at (-79.0, 45.5)
- added R35: 10K, spectrum3b:Passive, F.Cu at (-79.0, 49.5)
- added R36: 680, spectrum3b:Passive, F.Cu at (-79.0, 53.6)
- added R37: 1K, spectrum3b:Passive, F.Cu at (-63.5, -27.4)
- added R4: 470, spectrum3b:Passive, F.Cu at (-94.6, 13.1)
- added R42: 1K, spectrum3b:Passive, F.Cu at (-63.5, -23.3)
- added R43: 3K, spectrum3b:Passive, F.Cu at (-63.5, -19.3)
- added R44: 5K1, spectrum3b:Passive, F.Cu at (-63.5, -15.2)
- added R45: 1K, spectrum3b:Passive, F.Cu at (-63.5, -11.2)
- added R46: 1K, spectrum3b:Passive, F.Cu at (-63.5, -7.13)
- added R47: 1K, spectrum3b:Passive, F.Cu at (-63.5, -3.08)
- added R48: 2K2, spectrum3b:Passive, F.Cu at (-63.5, 0.97)
- added R49: 10K, spectrum3b:Passive, F.Cu at (-63.5, 5.02)
- added R5: 470, spectrum3b:Passive, F.Cu at (-94.6, 17.2)
- added R50: 4K7, spectrum3b:Passive, F.Cu at (-63.5, 9.07)
- added R51: 2K2, spectrum3b:Passive, F.Cu at (-63.5, 13.1)
- added R52: 2K2, spectrum3b:Passive, F.Cu at (-63.5, 17.2)
- added R53: 390R, spectrum3b:Passive, F.Cu at (-63.5, 21.2)
- added R54: 100K, spectrum3b:Passive, F.Cu at (-63.5, 25.3)
- added R55: 56, spectrum3b:Passive, F.Cu at (-63.5, 29.3)
- added R56: 1K, spectrum3b:Passive, F.Cu at (-63.5, 33.4)
- added R58: 1K, spectrum3b:Passive, F.Cu at (-63.5, 37.4)
- added R59: 1K8, spectrum3b:Passive, F.Cu at (-63.5, 41.4)
- added R6: 470, spectrum3b:Passive, F.Cu at (-94.6, 21.2)
- added R60: 68R, spectrum3b:Passive, F.Cu at (-63.5, 45.5)
- added R61: 15, spectrum3b:Passive, F.Cu at (-63.5, 49.5)
- added R62: 15, spectrum3b:Passive, F.Cu at (-63.5, 53.6)
- added R63: 1K, spectrum3b:Passive, F.Cu at (-47.9, -27.4)
- added R64: 15, spectrum3b:Passive, F.Cu at (-47.9, -23.3)
- added R65: 10K, spectrum3b:Passive, F.Cu at (-47.9, -19.3)
- added R66: 10K, spectrum3b:Passive, F.Cu at (-47.9, -15.2)
- added R67: 10K, spectrum3b:Passive, F.Cu at (-47.9, -11.2)
- added R68: 10K, spectrum3b:Passive, F.Cu at (-47.9, -7.13)
- added R69: 10K, spectrum3b:Passive, F.Cu at (-47.9, -3.08)
- added R7: 470, spectrum3b:Passive, F.Cu at (-94.6, 25.3)
- added R70: 220, spectrum3b:Passive, F.Cu at (-47.9, 0.97)
- added R71: 220, spectrum3b:Passive, F.Cu at (-47.9, 5.02)
- added R72: 10K, spectrum3b:Passive, F.Cu at (-47.9, 9.07)
- added R73: 1k, spectrum3b:Passive, F.Cu at (-47.9, 13.1)
- added R74: 10K, spectrum3b:Passive, F.Cu at (-47.9, 17.2)
- added R75: 10K, spectrum3b:Passive, F.Cu at (-47.9, 21.2)
- added R76: 1K, spectrum3b:Passive, F.Cu at (102.1, 75.3)
- added R77: 1K, spectrum3b:Passive, F.Cu at (102.1, 94.4)
- added R78: 470, spectrum3b:Passive, F.Cu at (102.1, 86.8)
- added R8: 470, spectrum3b:Passive, F.Cu at (-94.6, 29.3)
- added R9: 8k2, spectrum3b:Passive, F.Cu at (-94.6, 33.4)
- added T1: Coil, spectrum3b:Coil, F.Cu at (241.7, 58.6)
- added TV1: Modulator, spectrum3b:Modulator, F.Cu at (70.3, 42.9)
- added X1: 14Mhz, spectrum3b:X1, F.Cu at (99.8, 60.2)
- added X2: 4.43Mhz, spectrum3b:X2, F.Cu at (102.0, 64.6)
Routing:
- net (no net): track 24813.4 -> 14494.9 mm, vias 1325 -> 833
- net GND: track 0.00 -> 5520.4 mm, vias 0 -> 179
- net +5V: track 0.00 -> 1868.5 mm, vias 0 -> 146
- net Net-(TR8-C): track 0.00 -> 584.1 mm, vias 0 -> 31
- net +9V: track 0.00 -> 517.9 mm, vias 0 -> 16
- net -5V: track 0.00 -> 407.3 mm, vias 0 -> 25
- net Net-(IC14-R-Y_INPUT): track 0.00 -> 363.0 mm, vias 0 -> 19
- net -12VAC: track 0.00 -> 275.3 mm, vias 0 -> 18
- net VIDEO: track 0.00 -> 228.3 mm, vias 0 -> 7
- net Net-(TR2-C): track 0.00 -> 80.0 mm, vias 0 -> 9
- net Net-(IC14-CHROMA_BIAS): track 0.00 -> 73.7 mm, vias 0 -> 8
- net Net-(IC14-B-Y_INPUT): track 0.00 -> 62.1 mm, vias 0 -> 5
- net Net-(T1-AA): track 0.00 -> 61.5 mm, vias 0 -> 4
- net Net-(T1-AB): track 0.00 -> 59.2 mm, vias 0 -> 3
- net Net-(IC1-OSC): track 0.00 -> 54.4 mm, vias 0 -> 5
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Other:
- outline, holes or cut-outs redrawn
- board text added: "COMP"

Commit message: moved applied footprints
Parts:
- moved R78 162.2 mm to (-47.9, 25.3)
- moved LS1 111.7 mm to (345.6, 140.3)
- moved T1 92.5 mm to (334.2, 57.5)
- moved TV1 70.0 mm to (69.6, -27.1)
Changed lines of the file:
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@@
 	(footprint "spectrum3b:Speaker"
 		(layer "F.Cu")
-		(at 233.9048 141.204)
+		(at 345.6472 140.3169)
 		(property "Reference" "LS1"
 			(at 0 -0.5 0)
@@
 	(footprint "spectrum3b:Modulator"
 		(layer "F.Cu")
-		(at 70.2602 42.866)
+		(at 69.5607 -27.132)
 		(property "Reference" "TV1"
 			(at 0 -14.5 0)
@@
 	(footprint "spectrum3b:Coil"
 		(layer "F.Cu")
-		(at 241.677 58.6202)
+		(at 334.177 57.4842)
 		(property "Reference" "T1"
 			(at 0 -0.5 0)
@@
 	(footprint "spectrum3b:Passive"
 		(layer "F.Cu")
-		(at 102.11745 86.8087)
+		(at -47.93025 25.27)
 		(property "Reference" "R78"
 			(at 0.25 -0.05615 0)
